Commit message: added collisions, last training artifacts, changed torques for default

File: assets/go2/urdf/go2.urdf (robot description, URDF)
Before this commit: robot go2_description, 29 links, 28 joints
Links:
- link Head_lower: geometry collision sphere radius=0.047
- link Head_upper: geometry collision cylinder length=0.09 radius=0.05

Commit message: play around with torques

File: assets/go2/urdf/go2.urdf (robot description, URDF)
Before this commit: robot go2_description, 29 links, 28 joints
Links:
- link Head_lower: geometry 
- link Head_upper: geometry 

Commit message: fixed torques, added docker compose

File: assets/go2/urdf/go2.urdf (robot description, URDF)
Before this commit: robot go2_description, 29 links, 28 joints
Joints:
- joint FL_calf_joint: limit lower=-2.7227 upper=-0.83776 effort=35.55 velocity=20.07 -> lower=-2.7227 upper=-0.83776 effort=45.43 velocity=20.07
- joint FR_calf_joint: limit lower=-2.7227 upper=-0.83776 effort=35.55 velocity=20.07 -> lower=-2.7227 upper=-0.83776 effort=45.43 velocity=20.07
- joint RL_calf_joint: limit lower=-2.7227 upper=-0.83776 effort=35.55 velocity=20.07 -> lower=-2.7227 upper=-0.83776 effort=45.43 velocity=20.07
- joint RR_calf_joint: limit lower=-2.7227 upper=-0.83776 effort=35.55 velocity=20.07 -> lower=-2.7227 upper=-0.83776 effort=45.43 velocity=20.07
